Commit message: add Yummy

File: assets/Yummy_Robot/urdf/Yummy_Robot.urdf (robot description, URDF)
Before this commit: robot Yummy_Robot, 11 links, 10 joints
Links:
- link L0: geometry collision mesh filename=../meshes/L0.STL; visual mesh filename=../meshes/L0.STL
- link L1: geometry collision mesh filename=../meshes/L1.STL; visual mesh filename=../meshes/L1.STL
- link L2: geometry collision mesh filename=../meshes/L2.STL; visual mesh filename=../meshes/L2.STL
- link L3: geometry collision mesh filename=../meshes/L3.STL; visual mesh filename=../meshes/L3.STL
- link L4: geometry collision mesh filename=../meshes/L4.STL; visual mesh filename=../meshes/L4.STL
- link L5: geometry collision mesh filename=../meshes/L5.STL; visual mesh filename=../meshes/L5.STL
- link L6: geometry collision mesh filename=../meshes/L6.STL; visual mesh filename=../meshes/L6.STL
- link Lpicker1: geometry collision mesh filename=../meshes/Lpicker1.STL; visual mesh filename=../meshes/Lpicker1.STL
- link Lpicker2: geometry collision mesh filename=../meshes/Lpicker2.STL; visual mesh filename=../meshes/Lpicker2.STL
- link base_link: geometry collision mesh filename=../meshes/base_link.STL; visual mesh filename=../meshes/base_link.STL
- link camera: geometry collision mesh filename=../meshes/camera.STL; visual mesh filename=../meshes/camera.STL
